File: remote/remote.sch (KiCad schematic (older format))
At the start: 34 parts, among them J1 Conn_01x04, J2 Conn_01x05, SW1 SW_Push, SW2 SW_Push, SW3 SW_Push, SW4 SW_Push, U1 STM32F030F4Px, U2 RFM69CW-915MHZ

Commit message: Update layout for v1.1
Parts:
- removed C6: .1uF, Capacitor_SMD:C_0402_1005Metric, symbol Device:C
- removed C7: 1uF, Capacitor_SMD:C_0402_1005Metric, symbol Device:C
- removed J2: Conn_01x05, Connector_PinSocket_2.54mm:PinSocket_1x05_P2.54mm_Vertical, symbol Connector_Generic:Conn_01x05
- added J2: Conn_01x03, Connector_PinSocket_2.54mm:PinSocket_1x03_P2.54mm_Vertical, symbol Connector_Generic:Conn_01x03
- BT1: footprint Battery:BatteryHolder_Keystone_3008_1x2450 -> Battery:BatteryHolder_Keystone_3034_1x20mm
- H1, H2, H3, H4: footprint MountingHole:MountingHole_4.3mm_M4_ISO14580 -> MountingHole:MountingHole_3.2mm_M3
- R1: footprint Resistor_SMD:R_0805_2012Metric_Pad1.15x1.40mm_HandSolder -> Resistor_SMD:R_0805_2012Metric_Pad1.20x1.40mm_HandSolder
- SW1, SW2, SW3, SW4: LCSC C318888 -> C318889
Connections:
- net GND: now also J2.3 (Pin_3)
- net SERIAL_OUT: now also J2.1 (Pin_1)
- net VCC: now also J2.2 (Pin_2)
- no-connect marks 10 -> 8
Changed lines of the file:
@@
 F 0 "BT1" H 1768 6546 50  0000 L CNN
 F 1 "Battery_Cell" H 1768 6455 50  0000 L CNN
-F 2 "Battery:BatteryHolder_Keystone_3008_1x2450" V 1650 6510 50  0001 C CNN
+F 2 "Battery:BatteryHolder_Keystone_3034_1x20mm" V 1650 6510 50  0001 C CNN
 F 3 "~" V 1650 6510 50  0001 C CNN
 	1    1650 6450
@@
 F 2 "homebrew:SW_TACTILE_5.1MM_TS-1187A-C-D-B" H 6250 1100 50  0001 C CNN
 F 3 "~" H 6250 1100 50  0001 C CNN
-F 4 "C318888" H 6250 900 50  0001 C CNN "LCSC"
+F 4 "C318889" H 6250 900 50  0001 C CNN "LCSC"
 	1    6250 900
 	1    0    0    -1
@@
 	1200 1050 1600 1050
 Wire Wire Line
-	2250 1050 2650 1050
-Wire Wire Line
 	2000 750  2000 1150
 Wire Wire Line
@@
 	1900 750  1900 1150
 Connection ~ 1600 750
-$Comp
-L power:VCC #PWR013
-U 1 1 5F9FD268
-P 2950 750
-F 0 "#PWR013" H 2950 600 50  0001 C CNN
-F 1 "VCC" H 2967 923 50  0000 C CNN
-F 2 "" H 2950 750 50  0001 C CNN
-F 3 "" H 2950 750 50  0001 C CNN
-	1    2950 750
-	1    0    0    -1
-$EndComp
 $Comp
 L Device:R R2
@@
 SWDIO
 $Comp
-L Connector_Generic:Conn_01x05 J2
-U 1 1 5FA40358
-P 8700 2300
-F 0 "J2" H 8618 2717 50  0000 C CNN
-F 1 "Conn_01x05" H 8618 2626 50  0000 C CNN
-F 2 "Connector_PinSocket_2.54mm:PinSocket_1x05_P2.54mm_Vertical" H 8700 2300 50  0001 C CNN
-F 3 "~" H 8700 2300 50  0001 C CNN
-	1    8700 2300
-	-1   0    0    -1
-$EndComp
-NoConn ~ 8900 2200
-$Comp
 L power:GND #PWR024
 U 1 1 5FA448EF
@@
 L power:VCC #PWR026
 U 1 1 5FA45091
-P 9450 2300
-F 0 "#PWR026" H 9450 2150 50  0001 C CNN
-F 1 "VCC" H 9467 2473 50  0000 C CNN
-F 2 "" H 9450 2300 50  0001 C CNN
-F 3 "" H 9450 2300 50  0001 C CNN
-	1    9450 2300
-	1    0    0    -1
-$EndComp
-Wire Wire Line
-	8900 2100 9100 2100
-Wire Wire Line
-	9100 2100 9100 2000
-Wire Wire Line
-	9100 2000 9200 2000
-Wire Wire Line
-	9200 2000 9200 2050
-Wire Wire Line
-	9450 2300 8900 2300
-NoConn ~ 8900 2400
+P 9450 2400
+F 0 "#PWR026" H 9450 2250 50  0001 C CNN
+F 1 "VCC" H 9467 2573 50  0000 C CNN
+F 2 "" H 9450 2400 50  0001 C CNN
+F 3 "" H 9450 2400 50  0001 C CNN
+	1    9450 2400
+	1    0    0    -1
+$EndComp
+Wire Wire Line
+	9450 2400 8900 2400
 Text Label 9000 2500 0    50   ~ 0
 SERIAL_OUT
@@
 Text Notes 8650 1800 0    50   ~ 0
 Serial out
-Wire Wire Line
-	2000 750  2250 750
-$Comp
-L Device:C C6
-U 1 1 5FA64654
-P 2250 900
-F 0 "C6" H 2135 854 50  0000 R CNN
-F 1 ".1uF" H 2135 945 50  0000 R CNN
-F 2 "Capacitor_SMD:C_0402_1005Metric" H 2288 750 50  0001 C CNN
-F 3 "~" H 2250 900 50  0001 C CNN
-F 4 "C1525" H 2250 900 50  0001 C CNN "LCSC"
-	1    2250 900
-	1    0    0    1
-$EndComp
-Connection ~ 2250 750
 $Comp
 L Device:C C4
@@
 	1    0    0    1
 $EndComp
-Wire Wire Line
-	2250 750  2650 750
-$Comp
-L Device:C C7
-U 1 1 5FA71A82
-P 2650 900
-F 0 "C7" H 2535 854 50  0000 R CNN
-F 1 "1uF" H 2535 945 50  0000 R CNN
-F 2 "Capacitor_SMD:C_0402_1005Metric" H 2688 750 50  0001 C CNN
-F 3 "~" H 2650 900 50  0001 C CNN
-F 4 "C52923" H 2650 900 50  0001 C CNN "LCSC"
-	1    2650 900
-	1    0    0    1
-$EndComp
-Connection ~ 2650 750
-Wire Wire Line
-	2650 750  2950 750
 $Comp
 L Device:C C9
@@
 F 0 "H1" H 6159 6153 60  0000 L CNN
 F 1 "HOLE" H 6159 6047 60  0000 L CNN
-F 2 "MountingHole:MountingHole_4.3mm_M4_ISO14580" H 6050 6100 60  0001 C CNN
+F 2 "MountingHole:MountingHole_3.2mm_M3" H 6050 6100 60  0001 C CNN
 F 3 "" H 6050 6100 60  0001 C CNN
 	1    6050 6100
@@
 F 0 "H2" H 6159 6353 60  0000 L CNN
 F 1 "HOLE" H 6159 6247 60  0000 L CNN
-F 2 "MountingHole:MountingHole_4.3mm_M4_ISO14580" H 6050 6300 60  0001 C CNN
+F 2 "MountingHole:MountingHole_3.2mm_M3" H 6050 6300 60  0001 C CNN
 F 3 "" H 6050 6300 60  0001 C CNN
 	1    6050 6300
@@
 F 0 "H3" H 6159 6553 60  0000 L CNN
 F 1 "HOLE" H 6159 6447 60  0000 L CNN
-F 2 "MountingHole:MountingHole_4.3mm_M4_ISO14580" H 6050 6500 60  0001 C CNN
+F 2 "MountingHole:MountingHole_3.2mm_M3" H 6050 6500 60  0001 C CNN
 F 3 "" H 6050 6500 60  0001 C CNN
 	1    6050 6500
@@
 F 0 "H4" H 6159 6753 60  0000 L CNN
 F 1 "HOLE" H 6159 6647 60  0000 L CNN
-F 2 "MountingHole:MountingHole_4.3mm_M4_ISO14580" H 6050 6700 60  0001 C CNN
+F 2 "MountingHole:MountingHole_3.2mm_M3" H 6050 6700 60  0001 C CNN
 F 3 "" H 6050 6700 60  0001 C CNN
 	1    6050 6700
@@
 F 3 "" H 1200 1050 50  0001 C CNN
 	1    1200 1050
-	1    0    0    -1
-$EndComp
-Connection ~ 2650 1050
-$Comp
-L power:GND #PWR011
-U 1 1 5F865AF9
-P 2650 1050
-F 0 "#PWR011" H 2650 800 50  0001 C CNN
-F 1 "GND" H 2655 877 50  0000 C CNN
-F 2 "" H 2650 1050 50  0001 C CNN
-F 3 "" H 2650 1050 50  0001 C CNN
-	1    2650 1050
 	1    0    0    -1
 $EndComp
@@
 F 0 "R1" V 643 1350 50  0000 C CNN
 F 1 "DNP" V 734 1350 50  0000 C CNN
-F 2 "Resistor_SMD:R_0805_2012Metric_Pad1.15x1.40mm_HandSolder" V 780 1350 50  0001 C CNN
+F 2 "Resistor_SMD:R_0805_2012Metric_Pad1.20x1.40mm_HandSolder" V 780 1350 50  0001 C CNN
 F 3 "~" H 850 1350 50  0001 C CNN
 	1    850  1350
@@
 F 2 "homebrew:SW_TACTILE_5.1MM_TS-1187A-C-D-B" H 6250 2100 50  0001 C CNN
 F 3 "~" H 6250 2100 50  0001 C CNN
-F 4 "C318888" H 6250 1900 50  0001 C CNN "LCSC"
+F 4 "C318889" H 6250 1900 50  0001 C CNN "LCSC"
 	1    6250 1900
 	1    0    0    -1
@@
 F 2 "homebrew:SW_TACTILE_5.1MM_TS-1187A-C-D-B" H 6250 3100 50  0001 C CNN
 F 3 "~" H 6250 3100 50  0001 C CNN
-F 4 "C318888" H 6250 2900 50  0001 C CNN "LCSC"
+F 4 "C318889" H 6250 2900 50  0001 C CNN "LCSC"
 	1    6250 2900
 	1    0    0    -1
@@
 F 2 "homebrew:SW_TACTILE_5.1MM_TS-1187A-C-D-B" H 6250 4100 50  0001 C CNN
 F 3 "~" H 6250 4100 50  0001 C CNN
-F 4 "C318888" H 6250 3900 50  0001 C CNN "LCSC"
+F 4 "C318889" H 6250 3900 50  0001 C CNN "LCSC"
 	1    6250 3900
 	1    0    0    -1
@@
 Wire Wire Line
 	5700 3900 5750 3900
+$Comp
+L Connector_Generic:Conn_01x03 J2
+U 1 1 5FB57114
+P 8700 2400
+F 0 "J2" H 8618 2075 50  0000 C CNN
+F 1 "Conn_01x03" H 8618 2166 50  0000 C CNN
+F 2 "Connector_PinSocket_2.54mm:PinSocket_1x03_P2.54mm_Vertical" H 8700 2400 50  0001 C CNN
+F 3 "~" H 8700 2400 50  0001 C CNN
+	1    8700 2400
+	-1   0    0    1
+$EndComp
+Wire Wire Line
+	9200 2050 9200 2000
+Wire Wire Line
+	9200 2000 9050 2000
+Wire Wire Line
+	9050 2000 9050 2300
+Wire Wire Line
+	9050 2300 8900 2300
+Wire Wire Line
+	2000 750  1900 750
+Connection ~ 1900 750
 $EndSCHEMATC
